File: _restore_backup_2026-07-21T01-43-40-803/Pangotag_PCB.kicad_pcb (KiCad board)
At the start: 6 copper layers, 23 x 18 mm, 90 parts, among them CN2 POGOPIN_2X04_P2.54_M, IC1 TLV3691IDPFR, IC2 TLV3691IDPFR, J1 USB_C_Receptacle, J2 Conn_Coaxial, J3 USB_B_Mini, J4 USB_A, J5 Conn_01x02, P1 USB_C_Plug, Q1 PMX100UNZ, Q2 PMX100UNZ, Q3 PMX100UNZ, Q4 PMX100UNZ, SW1 SW_Push, U1 TPS62840YBGR, U11 AS6221T-AWLT, U13 TPS62840YBGR, U14 BMP581, U15 TMUX1575YCJR, U16 BMI270, U18 TPS62840YBGR, U3 SN74AUP1G08DPWR, U4 STM32U585OIYxQ, U5 TMUX1575YCJR, U6 MIA-M10Q, U7 LTC2941IDCB-1#TRMPBF, Y1 CM9V-T1A-32.768KHZ-7PF-20PPM-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

Commit message: layout done
Parts:
- moved U6 0.70 mm to (106.0, 53.7)
- moved C21 0.67 mm to (108.7, 51.2)
- moved U11 0.50 mm to (89.5, 47.0)
- moved C23 0.37 mm to (88.0, 47.1)
- moved U7 0.37 mm to (101.9, 52.8)
Routing:
- net GND: track 19.9 -> 0.00 mm
- net VDDA: track 19.7 -> 0.00 mm, vias 2 -> 0
- net Net-(Q4-D): track 5.93 -> 0.00 mm
- net VLXSMPS: track 4.83 -> 0.00 mm
- net Net-(Q3-D): track 4.54 -> 0.00 mm
- net Net-(Q2-D): track 3.61 -> 0.00 mm
- net +3V3: track 2.59 -> 0.00 mm, vias 1 -> 0
- net Net-(Q1-D): track 2.40 -> 0.00 mm
- net USBC_FUNCTION: vias 1 -> 0
Other:
- copper layers 6 -> 4
