File: Communication.kicad_sch (KiCad schematic)
At the start: 53 parts, among them IC1 TLV3691IDPFR, IC2 TLV3691IDPFR, J1 USB_C_Receptacle, J2 Conn_Coaxial, SW1 SW_Push, U11 AS6221T-AWLT, U14 BMP581, U15 TMUX1575YCJR, U16 BMI270, U3 SN74AUP1G08DPWR, U4 STM32U585OIYxQ, U5 TMUX1575YCJR, U6 MIA-M10Q, Y1 CM9V-T1A-32.768KHZ-7PF-20PPM-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

Commit message: Add V2: STM32U575 LQFP-64 tag board and ST-Link dongle
The tag moves from the 23 × 18 mm STM32U585 WLCSP-90 layout to a
31.94 × 27.18 mm, 6-layer board (Pangotag_PCB_LCSC_compat4.kicad_pcb) with
an LQFP-64 STM32U575, a MAX-M10S GNSS module, a 32 GB eMMC and parts that
JLCPCB stocks. Adds the USB-C debug dongle, the intermediate revisions, the
JLCPCB production files, the project footprint and symbol libraries, BOMs
and renders, plus a README.

Stops tracking KiCad lock files, the local-history folder and .DS_Store,
and ignores them along with large 3D exports.
Parts:
- removed C24: 100n, Capacitor_SMD:C_0201_0603Metric, symbol Device:C
- removed C25, C30: 10u, Capacitor_SMD:C_0201_0603Metric, symbol Device:C
- removed C32: 2.2u, Capacitor_SMD:C_0201_0603Metric, symbol Device:C
- removed C34: 4.7u, Capacitor_SMD:C_0201_0603Metric, symbol Device:C
- removed IC1, IC2: TLV3691IDPFR, TLV3691:TLV3691IDPFR, symbol TLV3691IDPFR:TLV3691IDPFR
- removed L5: 2.2u, Inductor_SMD:L_0201_0603Metric, symbol Device:L
- removed R12: 10k, Resistor_SMD:R_0201_0603Metric, symbol R_0603_US_2
- removed SW1: SW_Push, Button_Switch_SMD:SW_SPST_B3U-1000P, symbol Switch:SW_Push
- removed U11: AS6221T-AWLT, AS6221T:BGA6C40P2X3_102X150X52, symbol AS6221T-AWLT:AS6221T-AWLT
- removed U15, U5: TMUX1575YCJR, TMUX1575YCJR:PREYCJ0016-IPC_A, symbol TMUX1575:TMUX1575YCJR
- removed U3: SN74AUP1G08DPWR, SN74AUP1G08:DPW0005A_TEX, symbol 2026-07-17_04-06-15:SN74AUP1G08DPWR
- removed U4: STM32U585OIYxQ, Package_CSP:ST_WLCSP-90_4.2x3.95mm_Layout18x10_P0.4mm_Stagger, symbol MCU_ST_STM32U5:STM32U585OIYxQ
- removed U6: MIA-M10Q, Package_LGA:ublox_LGA-53_4.5x4.5mm_Layout9x9_P0.5mm, symbol RF_GPS:MIA-M10Q
- added C39, C40: 100n, Capacitor_SMD:C_0201_0603Metric, symbol Device:C
- added C4: 10n, Capacitor_SMD:C_0402_1005Metric, symbol Device:C
- added R5: 10, Resistor_SMD:R_0402_1005Metric, symbol Device:R_US
- added U1: 74AUP1G08GS_132, XSON6_SOT1202_NEX, symbol 74AUP1G08GS:74AUP1G08GS_132
- added U10, U9: TLV7031DPWR, easyeda2kicad:X2SON-4_L0.8-W0.8-P0.48-TL-A, symbol easyeda2kicad:TLV7031DPWR
- added U3: T117_C19284874, easyeda2kicad:TDFN-6_L2.0-W2.0-P0.65-TL-EP, symbol easyeda2kicad:T117_C19284874
- added U4: MAX-M10S, RF_GPS:ublox_MAX, symbol RF_GPS:MAX-M10S
- added U5: STM32U575RGTx, Package_QFP:LQFP-64_10x10mm_P0.5mm, symbol MCU_ST_STM32U5:STM32U575RGTx
- added U7: TMUX1511RSVR, easyeda2kicad:UTQFN-16_L2.6-W1.8-P0.40-BL, symbol easyeda2kicad:TMUX1511RSVR
- C22: footprint Capacitor_SMD:C_0201_0603Metric -> Capacitor_SMD:C_0402_1005Metric
- C31: value 2.2u -> 100n
- C33: value 100n -> 4.7u
- C35: value 100n -> 10u; footprint Capacitor_SMD:C_0201_0603Metric -> Capacitor_SMD:C_0402_1005Metric
- C37: value 1u -> 100n
- L1: value 100n -> 27n; footprint Inductor_SMD:L_0201_0603Metric -> Inductor_SMD:L_0402_1005Metric
Connections:
- net +1V8: now also C26.1, C27.1, C28.1, C31.1, C39.2, C40.2, U1.6 (VCC), U10.2 (VCC), U3.5 (VDD), U4.6 (V_BCKP), U4.7 (VCC_IO), U4.8 (VCC), U5.13 (VDDA), U5.19 (VDD), U5.32 (VDD), U5.64 (VDD), U7.16 (VDD), U9.2 (VCC); no longer C26.2, C27.2, C28.2, C33.2
- net +3V3: now also R5.1, U5.48 (VDDUSB); no longer L1.1
- net ACC_INT1: now also U5.14 (PA0)
- net ACC_INT2: now also U5.15 (PA1)
- net CC1: now also U9.4 (IN+)
- net CC2: now also U10.4 (IN+)
- net GND: now also C26.2, C27.2, C28.2, C33.2, C39.1, C4.2, C40.1, U1.3 (GND), U10.5 (VEE), U3.2 (GND), U3.4 (ADDR), U3.7 (EP), U4.1 (GND), U4.10 (GND), U4.12 (GND), U5.12 (VSSA), U5.18 (VSS), U5.31 (VSS), U5.47 (VSS), U5.63 (VSS), U7.8 (GND), U9.5 (VEE); no longer C26.1, C27.1, C28.1, C33.1
- net GPS_EXTINT: now also U4.5 (EXTINT), U5.11 (PC3)
- net I2C1_SCL: now also U3.1 (SCL), U4.17 (SCL), U5.29 (PB10)
- net I2C1_SDA: now also U3.6 (SDA), U4.16 (SDA), U5.35 (PB14)
- net LED1: now also U5.27 (PB1)
- net LED2: now also U5.26 (PB0)
- net LED3: now also U5.23 (PA7)
- net LED4: now also U5.22 (PA6)
- net NRST: now also U5.7 (NRST), U7.13 (D4)
- net OSC32_IN: now also U5.3 (PC14)
- net OSC32_OUT: now also U5.4 (PC15)
- net PRS_INT: now also U5.9 (PC1)
- net RF_IN: now also U4.11 (RF_IN)
- net SDMMC1_CK: now also U5.53 (PC12)
- net SDMMC1_CMD: now also U5.54 (PD2)
- net SDMMC1_D0: now also U5.39 (PC8)
- net SDMMC1_D1: now also U5.40 (PC9)
- net SDMMC1_D2: now also U5.51 (PC10)
- net SDMMC1_D3: now also U5.52 (PC11)
- net SWCLK: now also U5.49 (PA14), U7.3 (D1)
- net SWDIO: now also U5.46 (PA13), U7.6 (D2)
- net SWO: now also U5.55 (PB3), U7.9 (D3)
- net Timepulse: now also U4.4 (TIMEPULSE), U5.10 (PC2)
- net USART1_RX: now also U4.2 (TXD), U5.43 (PA10)
- net USART1_TX: now also U4.3 (RXD), U5.58 (PB6)
- net USBC_FUNCTION: now also U1.4 (Y), U7.1 (SEL1), U7.11 (SEL3), U7.15 (SEL4), U7.4 (SEL2)
- net USB_OTG_VBUS: now also U5.42 (PA9)
- net VBAT/3: now also U5.8 (PC0)
- net at R21.2, R22.1: now also U10.3 (IN-), U9.3 (IN-)
- net at J1.B3 (TX2-): now also U7.5 (S2)
- net at J1.B11 (RX1+): now also U7.10 (S3)
- net at J1.A2 (TX1+): now also U7.2 (S1)
- net at J1.B8 (SBU2): now also U7.14 (S4)
- net USB_OTG_FS_DM renamed USB_OTG_FS_D-
- net USB_OTG_FS_D-: now also U5.44 (PA11)
- net USB_OTG_FS_DP renamed USB_OTG_FS_D+
- net USB_OTG_FS_D+: now also U5.45 (PA12)
- new net: U1.2 (A), U10.1 (OUT)
- new net: C4.1, L1.1, R5.2
- new net: C33.1, U5.30 (VCAP)
- new net: U1.1 (B), U9.1 (OUT)
Other:
- note added: "2 uA at 1 meas/s"
- note added: "Temperature Sensor (0x40)"
- note removed: "6 uA (4 Hz) estimating about 1.575 uA for 1 Hz (with 36 ms active time for conversion) 0.1 uA (standby)"
- note removed: "Reset Button"
- note removed: "Temperature Sensor (0x58)"
- moved on the sheet: C23, L1, R15, R16, R21, R22
