File: LEDs.kicad_sch (KiCad schematic)
At the start: 12 parts, among them Q1 PMX100UNZ, Q2 PMX100UNZ, Q3 PMX100UNZ, Q4 PMX100UNZ

Commit message: Add V2: STM32U575 LQFP-64 tag board and ST-Link dongle
The tag moves from the 23 × 18 mm STM32U585 WLCSP-90 layout to a
31.94 × 27.18 mm, 6-layer board (Pangotag_PCB_LCSC_compat4.kicad_pcb) with
an LQFP-64 STM32U575, a MAX-M10S GNSS module, a 32 GB eMMC and parts that
JLCPCB stocks. Adds the USB-C debug dongle, the intermediate revisions, the
JLCPCB production files, the project footprint and symbol libraries, BOMs
and renders, plus a README.

Stops tracking KiCad lock files, the local-history folder and .DS_Store,
and ignores them along with large 3D exports.
Parts:
- D1, D2, D3, D4: footprint LED_SMD:LED_0201_0603Metric -> LED_SMD:LED_0603_1608Metric
Changed lines of the file:
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@@
 			)
 		)
-		(property "Footprint" "LED_SMD:LED_0201_0603Metric"
+		(property "Footprint" "LED_SMD:LED_0603_1608Metric"
 			(at 73.66 57.15 0)
 			(hide yes)
@@
 			)
 		)
-		(property "Footprint" "LED_SMD:LED_0201_0603Metric"
+		(property "Footprint" "LED_SMD:LED_0603_1608Metric"
 			(at 184.15 58.42 0)
 			(hide yes)
@@
 			)
 		)
-		(property "Footprint" "LED_SMD:LED_0201_0603Metric"
+		(property "Footprint" "LED_SMD:LED_0603_1608Metric"
 			(at 224.79 57.15 0)
 			(hide yes)
@@
 			)
 		)
-		(property "Footprint" "LED_SMD:LED_0201_0603Metric"
+		(property "Footprint" "LED_SMD:LED_0603_1608Metric"
 			(at 132.08 57.15 0)
 			(hide yes)
