File: st-link_conn.kicad_sch (KiCad schematic)
At the start: 10 parts, among them CN2 POGOPIN_2X04_P2.54_M, J3 USB_B_Mini, J4 USB_A, P1 USB_C_Plug, U18 TPS62840YBGR

Commit message: Add V2: STM32U575 LQFP-64 tag board and ST-Link dongle
The tag moves from the 23 × 18 mm STM32U585 WLCSP-90 layout to a
31.94 × 27.18 mm, 6-layer board (Pangotag_PCB_LCSC_compat4.kicad_pcb) with
an LQFP-64 STM32U575, a MAX-M10S GNSS module, a 32 GB eMMC and parts that
JLCPCB stocks. Adds the USB-C debug dongle, the intermediate revisions, the
JLCPCB production files, the project footprint and symbol libraries, BOMs
and renders, plus a README.

Stops tracking KiCad lock files, the local-history folder and .DS_Store,
and ignores them along with large 3D exports.
Parts:
- removed J4: USB_A, Connector_USB:USB_A_Molex_48037-2200_Horizontal, symbol Connector:USB_A
- removed P1: USB_C_Plug, Connector_USB:USB_C_Plug_ShenzhenJingTuoJin_918-118A2021Y40002_Vertical, symbol Connector:USB_C_Plug
- removed R14, R5: 56k, Resistor_SMD:R_0201_0603Metric, symbol Device:R_US
- added D+1, D-1, GND1, ID1, VBUS1: MountingHole_Pad, TestPoint:TestPoint_Pad_1.5x1.5mm, symbol Mechanical:MountingHole_Pad
- added J4: UP32-C-F-G-FL-3-P24-TR, easyeda2kicad:USB-TH-TYPE-C_00702-UCAM002-X, symbol UP32-C-F-G-FL-3-P24-TR:UP32-C-F-G-FL-3-P24-TR
- added R10, R17: 56k, Resistor_SMD:R_0201_0603Metric, symbol Device:R_US
- added R12: 10k, Resistor_SMD:R_0201_0603Metric, symbol R_0603_US_2
- added SW1: SW_Push, Button_Switch_SMD:SW_SPST_B3U-1000P, symbol Switch:SW_Push
- C19: footprint Capacitor_SMD:C_0201_0603Metric -> Capacitor_SMD:C_0402_1005Metric
- CN2: footprint Connector_PinSocket_2.54mm:PinSocket_2x03_P2.54mm_Vertical_SMD -> Connector_PinHeader_2.54mm:PinHeader_2x03_P2.54mm_Vertical
- L4: footprint Inductor_SMD:L_0201_0603Metric -> Inductor_SMD:L_0805_2012Metric
Connections:
- net +1V8_2: now also R12.1
- net NRST_OUT: now also J4.A8 (SBU1), J4.B8 (SBU2), R12.2, SW1.1
- net SWCLK_OUT: now also J4.A2 (SSTXP1), J4.B2 (SSTXP2)
- net SWDIO_OUT: now also J4.A3 (SSTXN1), J4.B3 (SSTXN2)
- net SWO_OUT: now also J4.A11 (SSRXP2), J4.B11 (SSRXP1)
- net VBUS_DONGLE: now also J4.A4 (VBUS_1), J4.A9 (VBUS_2), J4.B4 (VBUS_3), J4.B9 (VBUS_4), R10.1, R17.1, VBUS1.1
- net ST_D-: now reaches J3.2 (D-)
- net ST_D-: now also D-1.1
- net ST_D+: now reaches J3.3 (D+)
- net ST_D+: now also D+1.1
- net at J3.4 (ID): now also ID1.1
- net GND renamed GND2
- net GND2: now also GND1.1, J4.A1 (GND_1), J4.A12 (GND_2), J4.B1 (GND_3), J4.B12 (GND_4), J4.MH1, J4.MH2, SW1.2
- new net: J4.A5 (CC1), R10.2
- new net: J4.B5 (CC2), R17.2
Other:
- note added: "Attach original male-male USB-A to Mini-B cable here"
- note added: "Reset Button"
- note added: "Solder short mini-B cable onto this to connect to ST-Link"
- note removed: "Attach female-male USB-A to Mini-B dongle here that goes into the ST-Link"
- note removed: "Attach male-male USB-A to Mini-B cable here"
